Commit message: 开源 1.0定版

File: src/Piper_ros/src/piper_description/urdf/piper_description.urdf (robot description, URDF)
Before this commit: robot piper_description, 9 links, 8 joints
Links:
- added link gripper_base, mass 0.145318531013916; collision mesh filename=/home/ppn/questVR_ws/src/Piper_ros/src/piper_description/me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; visual mesh filename=/home/ppn/questVR_ws/src/Piper_ros/src/piper_description/me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
- link base_link: mass 0.162352169522719 -> 0.333893486740112; geometry collision mesh filename=/home/ppn/questVR_ws/src/Piper_ros/src/piper_description/me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; visual mesh filename=/home/ppn/questVR_ws/src/Piper_ros/src/piper_description/me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
- link link1: mass 0.0978679932242825 -> 0.215052383265765; geometry collision mesh filename=/home/ppn/questVR_ws/src/Piper_ros/src/piper_description/me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; visual mesh filename=/home/ppn/questVR_ws/src/Piper_ros/src/piper_description/me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
- link link2: mass 0.289571136953082 -> 0.463914239236335; geometry collision mesh filename=/home/ppn/questVR_ws/src/Piper_ros/src/piper_description/me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; visual mesh filename=/home/ppn/questVR_ws/src/Piper_ros/src/piper_description/me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
- link link3: mass 0.290583243387798 -> 0.219942452993132; geometry collision mesh filename=/home/ppn/questVR_ws/src/Piper_ros/src/piper_description/me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; visual mesh filename=/home/ppn/questVR_ws/src/Piper_ros/src/piper_description/me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
- link link4: mass 0.127087348341362 -> 0.131814339939458; geometry collision mesh filename=/home/ppn/questVR_ws/src/Piper_ros/src/piper_description/me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; visual mesh filename=/home/ppn/questVR_ws/src/Piper_ros/src/piper_description/me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
- link link5: mass 0.144711242639456 -> 0.134101341225523; geometry collision mesh filename=/home/ppn/questVR_ws/src/Piper_ros/src/piper_description/me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; visual mesh filename=/home/ppn/questVR_ws/src/Piper_ros/src/piper_description/me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
- link link6: mass 0.150196493124859 -> 0.00699089613564366; geometry collision mesh filename=/home/ppn/questVR_ws/src/Piper_ros/src/piper_description/me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; visual mesh filename=/home/ppn/questVR_ws/src/Piper_ros/src/piper_description/me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
- link link7: mass 0.0264822923452701 -> 0.0303534920715906; geometry collision mesh filename=/home/ppn/questVR_ws/src/Piper_ros/src/piper_description/me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; visual mesh filename=/home/ppn/questVR_ws/src/Piper_ros/src/piper_description/me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
- link link8: mass 0.0264822021416581 -> 0.0303534920715904; geometry collision mesh filename=/home/ppn/questVR_ws/src/Piper_ros/src/piper_description/me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; visual mesh filename=/home/ppn/questVR_ws/src/Piper_ros/src/piper_description/me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
Joints:
- added joint joint6_to_gripper_base: type fixed, parent link6, child gripper_base, origin xyz=0 0 0 rpy=0 0 0
- joint joint1: limit lower=-2.618 upper=2.618 effort=100 velocity=3 -> lower=-2.618 upper=2.168 effort=100 velocity=5; origin xyz=0 0 0.123 rpy=0 0 -1.5708 -> xyz=0 0 0.123 rpy=0 0 0
- joint joint2: limit lower=0 upper=3.14 effort=100 velocity=3 -> lower=0 upper=3.14 effort=100 velocity=5; origin xyz=0 0 0 rpy=1.5708 -0.10095 -1.5708 -> xyz=0 0 0 rpy=1.5708 -0.10095 -3.1416
- joint joint3: limit lower=-2.697 upper=0 effort=100 velocity=3 -> lower=-2.967 upper=0 effort=100 velocity=5; origin xyz=0.28503 0 0 rpy=0 0 1.3826 -> xyz=0.28503 0 0 rpy=0 0 -1.759
- joint joint4: limit lower=-1.832 upper=1.832 effort=100 velocity=3 -> lower=-1.745 upper=1.745 effort=100 velocity=5; origin xyz=0.021984 0.25075 0 rpy=-1.5708 0 0 -> xyz=-0.021984 -0.25075 0 rpy=1.5708 0 0
- joint joint5: limit lower=-1.22 upper=1.22 effort=100 velocity=3 -> lower=-1.22 upper=1.22 effort=100 velocity=5; origin xyz=0 0 0 rpy=1.5708 0 0 -> xyz=0 0 0 rpy=-1.5708 0 0
- joint joint6: axis 0 0 -1 -> 0 0 1; limit lower=-3.14 upper=3.14 effort=100 velocity=3 -> lower=-2.0944 upper=2.0944 effort=100 velocity=3; origin xyz=0 0.091 0.0014165 rpy=-1.5708 -1.5708 0 -> xyz=8.8259E-05 -0.091 0 rpy=1.5708 0 0
- joint joint7: axis 0 0 -1 -> 0 0 1; limit lower=0 upper=0.04 effort=10 velocity=1 -> lower=0 upper=0.035 effort=10 velocity=1; origin xyz=0 0 0.13503 rpy=1.5708 0 1.5708 -> xyz=0 0 0.1358 rpy=1.5708 0 0; parent link6 -> gripper_base
- joint joint8: axis 0 0 1 -> 0 0 -1; limit lower=-0.04 upper=0 effort=10 velocity=1 -> lower=-0.035 upper=0 effort=10 velocity=1; origin xyz=0 0 0.13503 rpy=-1.5708 0 1.5708 -> xyz=0 0 0.1358 rpy=1.5708 0 -3.1416; parent link6 -> gripper_base

Commit message: update piper urdf joint1 limit

File: src/Piper_ros/src/piper_description/urdf/piper_description.urdf (robot description, URDF)
Before this commit: robot piper_description, 10 links, 9 joints
Links:
- link base_link: geometry collision mesh filename=/home/agilex/questVR_ws/src/Piper_ros/src/piper_description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; visual mesh filename=/home/agilex/questVR_ws/src/Piper_ros/src/piper_description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
- link gripper_base: geometry collision mesh filename=/home/agilex/questVR_ws/src/Piper_ros/src/piper_description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; visual mesh filename=/home/agilex/questVR_ws/src/Piper_ros/src/piper_description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
- link link1: geometry collision mesh filename=/home/agilex/questVR_ws/src/Piper_ros/src/piper_description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; visual mesh filename=/home/agilex/questVR_ws/src/Piper_ros/src/piper_description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
- link link2: geometry collision mesh filename=/home/agilex/questVR_ws/src/Piper_ros/src/piper_description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; visual mesh filename=/home/agilex/questVR_ws/src/Piper_ros/src/piper_description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
- link link3: geometry collision mesh filename=/home/agilex/questVR_ws/src/Piper_ros/src/piper_description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; visual mesh filename=/home/agilex/questVR_ws/src/Piper_ros/src/piper_description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
- link link4: geometry collision mesh filename=/home/agilex/questVR_ws/src/Piper_ros/src/piper_description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; visual mesh filename=/home/agilex/questVR_ws/src/Piper_ros/src/piper_description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
- link link5: geometry collision mesh filename=/home/agilex/questVR_ws/src/Piper_ros/src/piper_description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; visual mesh filename=/home/agilex/questVR_ws/src/Piper_ros/src/piper_description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
- link link6: geometry collision mesh filename=/home/agilex/questVR_ws/src/Piper_ros/src/piper_description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; visual mesh filename=/home/agilex/questVR_ws/src/Piper_ros/src/piper_description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
- link link7: geometry collision mesh filename=/home/agilex/questVR_ws/src/Piper_ros/src/piper_description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; visual mesh filename=/home/agilex/questVR_ws/src/Piper_ros/src/piper_description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
- link link8: geometry collision mesh filename=/home/agilex/questVR_ws/src/Piper_ros/src/piper_description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; visual mesh filename=/home/agilex/questVR_ws/src/Piper_ros/src/piper_description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
Joints:
- joint joint1: limit lower=-2.618 upper=2.168 effort=100 velocity=5 -> lower=-2.618 upper=2.618 effort=100 velocity=5
